File: a2m2010.kicad_sch (KiCad schematic)
At the start: 176 parts, among them IC301 TCA1170N, IC601 L78S15CV, J1 Conn_Coaxial, Q101 2SC1815, Q102 2SA1015, Q104 2sa1015, Q105 2SC945CY, Q201 2N2222A, Q202 BF256, Q203 2SC1815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

Commit message: Added PDF of Schematic
Other:
- company: (none) -> A Thousand Projects
- title: (none) -> Apple Monitor II A2M2010 Schematic
- moved on the sheet: C101, C102, C103, C108, C109, C110, C111, C112, C133, C202, C203, C206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
